File: Tbogg_Sensor_Pkg_PCB/LoRa_Module.kicad_sch (KiCad schematic)
At the start: 9 parts, among them J201 Conn_01x04, J202 Conn_Coaxial, U201 LoRa-E5

Commit message: Finish design
Parts:
- removed C203, C204: NC, Capacitor_SMD:C_1206_3216Metric_Pad1.33x1.80mm_HandSolder, symbol Device:C
- removed J201: Conn_01x04, Connector_PinHeader_2.54mm:PinHeader_1x04_P2.54mm_Vertical, symbol Connector_Generic:Conn_01x04
- removed L201: 0, Inductor_SMD:L_1206_3216Metric_Pad1.42x1.75mm_HandSolder, symbol Device:L
- removed TP201: TestPoint, TestPoint:TestPoint_Pad_D3.0mm, symbol Connector:TestPoint
- added J307: Conn_01x02, Connector_PinHeader_2.54mm:PinHeader_1x02_P2.54mm_Vertical, symbol Connector_Generic:Conn_01x02
Connections:
- net LORA_UART_MISO: now also J307.1 (Pin_1)
- net LORA_UART_MOSI: now also J307.2 (Pin_2)
- net at J202.1 (In): now also U201.15 (RFIO)
- no-connect marks 19 -> 20
