File: Tbogg_Sensor_Pkg_PCB/ModulesA.kicad_sch (KiCad schematic)
At the start: 16 parts, among them J401 100k_Thermistor, J402 100k_Thermistor, U401 GY-NEO6MV2-Module, U403 STDS75DS2F

Commit message: Finish design
Parts:
- removed H403, H404, H407, H408: MountingHole, MountingHole:MountingHole_2mm, symbol Mechanical:MountingHole
- added J403: Conn_01x04, Connector_PinHeader_2.54mm:PinHeader_1x04_P2.54mm_Vertical, symbol Connector_Generic:Conn_01x04
Connections:
- net +3V3: now also J403.1 (Pin_1)
- net GND: now also J403.2 (Pin_2)
- net SCL: now also J403.3 (Pin_3)
- net SDA: now also J403.4 (Pin_4)
Other:
- note added: "Accelerometer Module"
