File: Tbogg_Sensor_Pkg_PCB/Power.kicad_sch (KiCad schematic)
At the start: 11 parts, among them J301 Conn_01x02, J302 Conn_01x04, J303 Conn_01x04, J304 Screw_Terminal_01x02, J305 Screw_Terminal_01x02, J306 Conn_01x04, J307 Conn_01x02, J308 Screw_Terminal_01x02, SW301 SW_SPDT

Commit message: Finish design
Parts:
- removed J301, J307: Conn_01x02, Connector_PinHeader_2.54mm:PinHeader_1x02_P2.54mm_Vertical, symbol Connector_Generic:Conn_01x02
- removed J302, J306: Conn_01x04, Connector_PinHeader_2.54mm:PinHeader_1x04_P2.54mm_Vertical, symbol Connector_Generic:Conn_01x04
Connections:
- net +3V3: no longer J303.1 (Pin_1), J303.2 (Pin_2)
- net GND: now also J303.1 (Pin_1), J303.2 (Pin_2)
Other:
- note removed: "Don't use this connector for balloon"
