File: Tbogg_Sensor_Pkg_PCB/Tbogg_Sensor_Pkg_PCB.kicad_sch (KiCad schematic)
At the start: 0 parts

Commit message: Add base from other project
Parts:
- added C101: 10u, Capacitor_SMD:C_1206_3216Metric_Pad1.33x1.80mm_HandSolder, symbol Device:C
- added D101, D102, D103, D104: LED, LED_SMD:LED_1206_3216Metric_Pad1.42x1.75mm_HandSolder, symbol Device:LED
- added H101, H102, H103, H104: MountingHole_Pad, MountingHole:MountingHole_3.2mm_M3_DIN965_Pad, symbol Mechanical:MountingHole_Pad
- added J101: Conn_01x04, Connector_PinHeader_2.54mm:PinHeader_1x04_P2.54mm_Vertical, symbol Connector_Generic:Conn_01x04
- added R101, R102: 4.7k, Resistor_SMD:R_1206_3216Metric_Pad1.30x1.75mm_HandSolder, symbol Device:R
- added R103: 3.3k, Resistor_SMD:R_1206_3216Metric_Pad1.30x1.75mm_HandSolder, symbol Device:R
- added R104, R105, R106: 1k, Resistor_SMD:R_1206_3216Metric_Pad1.30x1.75mm_HandSolder, symbol Device:R
- added U101: ESP32-Module-30Pin, 00 This Project Symbol Lib:ESP32-Module-30Pin, symbol 00_This_Project_Symbol_Lib:ESP32-Module-30Pin
Connections:
- new net: R105.1, U101.8 (D5/VSPI_CS0)
- new net: D103.2 (A), R105.2
- new net: D101.2 (A), R103.2
- new net: D102.2 (A), R104.2
- new net: J101.1 (Pin_1), U101.10 (D19/VSPI_MISO)
- new net: J101.2 (Pin_2), U101.15 (D23/VSPI_MOSI)
- new net: C101.1, U101.16 (EN)
- new net: J101.4 (Pin_4), U101.20 (D35/ADC1_CH7)
- new net: J101.3 (Pin_3), U101.25 (D27/ADC2_CH7/TOUCH7)
- new net: D104.2 (A), R106.2
- new net +3V3: R101.1, R102.1, R104.1, U101.1 (3V3)
- new net +BATT: R103.1
- new net BATT_SENSE: U101.19 (D34/ADC1_CH6)
- new net DHT_DATA: U101.24 (D26/ADC2_CH9/DAC2)
- new net GND: C101.2, D101.1 (K), D102.1 (K), D103.1 (K), D104.1 (K), H101.1, H102.1, H103.1, H104.1, U101.2 (GND_2), U101.29 (GND_1)
- new net GPS_UART_MISO: U101.5 (D4/ADC2_CH0/TOUCH0)
- new net GPS_UART_MOSI: U101.28 (D13/ADC2_CH4/TOUCH4/HSPI_MOSI)
- new net HEATER_EN: R106.1, U101.26 (D14/ADC2_CH6/TOUCH6/HSPI_CLK)
- new net LORA_UART_MISO: U101.6 (RX2/D16)
- new net LORA_UART_MOSI: U101.7 (TX2/D17)
- new net MCU_VIN: U101.30 (VIN)
- new net RTF_SWITCH: U101.9 (D18/VSPI_CLK)
- new net SCL: R101.2, U101.14 (D22/I2C_SCL)
- new net SDA: R102.2, U101.11 (D21/I2C_SDA)
- new net TEMP_SENSE_1: U101.22 (D33/ADC1_CH5/TOUCH8)
- new net TEMP_SENSE_2: U101.21 (D32/ADC1_CH4/TOUCH9)
- new net TEMP_V+: U101.23 (D25/ADC2_CH8/DAC1)
- no-connect marks 0 -> 7
Other:
- added sheet LoRa_Module (LoRa_Module.kicad_sch)
- added sheet ModulesA (ModulesA.kicad_sch)
- added sheet Power (Power.kicad_sch)
- note added: "D2 = Onb. LED"
- note added: "DNU D12"
- note added: "GP Breakout"
- note added: "I2C Pullups"
- note added: "LoRa Module"
- note added: "Modules A"
- note added: "Power"

Commit message: Finish design
Parts:
- removed D101, D102, D103, D104: LED, LED_SMD:LED_1206_3216Metric_Pad1.42x1.75mm_HandSolder, symbol Device:LED
- removed R103: 3.3k, Resistor_SMD:R_1206_3216Metric_Pad1.30x1.75mm_HandSolder, symbol Device:R
- removed R104, R105, R106: 1k, Resistor_SMD:R_1206_3216Metric_Pad1.30x1.75mm_HandSolder, symbol Device:R
Connections:
- net STRAIN_SENSE: now reaches U101.17 (VP/ADC1_CH0)
- net DHT_DATA: no longer names the net of U101.24 (D26/ADC2_CH9/DAC2)
- net HEATER_EN: no longer names the net of U101.26 (D14/ADC2_CH6/TOUCH6/HSPI_CLK)
- net RTF_SWITCH: no longer names the net of U101.9 (D18/VSPI_CLK)
- no-connect marks 7 -> 9
Other:
- added sheet Strain_Sensor (Strain_Sensor.kicad_sch)
