File: Tbogg_Sensor_Pkg_PCB/Tbogg_Sensor_Pkg_PCB.kicad_pcb (KiCad board)
At the start: 2 copper layers, 52 x 67 mm, 48 parts, among them J101 Conn_01x04, J202 Conn_Coaxial, J203 Conn_01x02, J303 Conn_01x04, J304 Screw_Terminal_01x02, J305 Screw_Terminal_01x02, J308 Screw_Terminal_01x02, J401 100k_Thermistor, J402 100k_Thermistor, J403 Conn_01x04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

Commit message: Tiny reroutes, labels
Parts:
- C501, C502, R503, U501: moved to F.Cu
- moved R102 10.1 mm to (74.5, 53.3)
- moved R101 10.1 mm to (74.5, 57.0)
- moved U403 10.1 mm to (80.6, 55.4)
- moved R503 9.29 mm to (93.3, 67.5)
- moved C501 6.67 mm to (94.6, 62.2), turned to 180 degrees
- moved C502 6.03 mm to (101.0, 62.2), turned to 180 degrees
- moved U501 2.91 mm to (99.4, 67.6), turned to 0 degrees
Routing:
- net SCL: track 81.0 -> 56.7 mm, vias 0 -> 1
- net +3V3: track 28.2 -> 35.3 mm, vias 4 -> 8
- net Net-(R505-Pad1): track 15.0 -> 20.7 mm, vias 2 -> 1
- net /Strain_Sensor/IN+: track 22.9 -> 28.3 mm
- net GND: track 8.36 -> 3.12 mm, vias 20 -> 17
- net MCU_VIN: track 37.4 -> 42.6 mm
- net SDA: track 52.8 -> 47.9 mm
- net /Strain_Sensor/V_REF: track 19.1 -> 15.6 mm
- net TEMP_V+: track 50.3 -> 51.6 mm
- net /Strain_Sensor/IN-: track 26.2 -> 27.0 mm, vias 0 -> 1
Other:
- board text added: "Accelerometer"
- board text added: "GNCTR 2024 Rev 1 Sensor Board"
- board text added: "Strain Gauge"
- board text added: "Top=GND Bottom=3V3 Edge Cuts: X: 104 - 52 = 52mm Y: 106 - 39 = 97mm Holes: M3, inset by 5mm"
- board text removed: "Motion ^"
- board text removed: "Top=GND Bottom=3V3"
