File: Tbogg_Sensor_Pkg_PCB/Tbogg_Sensor_Pkg_PCB.kicad_pcb (KiCad board)
At the start: 2 copper layers, 52 x 67 mm, 48 parts, among them J101 Conn_01x04, J202 Conn_Coaxial, J203 Conn_01x02, J303 Conn_01x04, J304 Screw_Terminal_01x02, J305 Screw_Terminal_01x02, J308 Screw_Terminal_01x02, J401 100k_Thermistor, J402 100k_Thermistor, J403 Conn_01x04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

Commit message: Comments updates
Other:
- board text added: "Top=GND Bottom=3V3 Edge Cuts: X: 104 - 52 = 52mm Y: 106 - 39 = 97mm USB port is centered, basically. Holes: M3, inset by 5mm"
- board text removed: "Top=GND Bottom=3V3 Edge Cuts: X: 104 - 52 = 52mm Y: 106 - 39 = 97mm Holes: M3, inset by 5mm"
Changed lines of the file:
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@@
     (effects (font (size 1 1) (thickness 0.15)) (justify left bottom))
   )
-  (gr_text "Top=GND\nBottom=3V3\n\nEdge Cuts:\nX: 104 - 52 = 52mm\nY: 106 - 39 = 97mm\n\nHoles: M3, inset by 5mm" (at 111.252 37.084) (layer "Cmts.User")
+  (gr_text "Top=GND\nBottom=3V3\n\nEdge Cuts:\nX: 104 - 52 = 52mm\nY: 106 - 39 = 97mm\n\nUSB port is centered, basically.\n\nHoles: M3, inset by 5mm" (at 111.252 37.084) (layer "Cmts.User")
     (effects (font (size 1 1) (thickness 0.15)) (justify left bottom))
   )

Commit message: Fix enclosure dimension on PCB comments layer
Other:
- board text added: "Top=GND Bottom=3V3 Edge Cuts: X: 104 - 52 = 52mm Y: 106 - 39 = 67mm Holes: M3, inset by 5mm"
- board text removed: "Top=GND Bottom=3V3 Edge Cuts: X: 104 - 52 = 52mm Y: 106 - 39 = 97mm USB port is centered, basically. Holes: M3, inset by 5mm"
Changed lines of the file:
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@@
     (effects (font (size 1 1) (thickness 0.15)) (justify left bottom))
   )
-  (gr_text "Top=GND\nBottom=3V3\n\nEdge Cuts:\nX: 104 - 52 = 52mm\nY: 106 - 39 = 97mm\n\nUSB port is centered, basically.\n\nHoles: M3, inset by 5mm" (at 111.252 37.084) (layer "Cmts.User")
+  (gr_text "Top=GND\nBottom=3V3\n\nEdge Cuts:\nX: 104 - 52 = 52mm\nY: 106 - 39 = 67mm\n\nHoles: M3, inset by 5mm" (at 111.252 37.084) (layer "Cmts.User")
     (effects (font (size 1 1) (thickness 0.15)) (justify left bottom))
   )
